Commit message: add aubo_i5 config file

File: aubo_description/urdf/aubo_i5L.urdf (robot description, URDF)
Before this commit: robot aubo_i5L_robot, 13 links, 12 joints
Links:
- link base_link: geometry collision mesh filename=package://aubo_description/meshes/aubo_i5l/base_link.STL; visual mesh filename=package://aubo_description/meshes/aubo_i5l/base_link.STL
- link f1_Link: geometry collision mesh filename=package://aubo_description/meshes/aubo_i5l/f1_Link.STL; visual mesh filename=package://aubo_description/meshes/aubo_i5l/f1_Link.STL
- link foreArm_Link: geometry collision mesh filename=package://aubo_description/meshes/aubo_i5l/foreArm_Link.STL; visual mesh filename=package://aubo_description/meshes/aubo_i5l/foreArm_Link.STL
- link s_Link: geometry collision mesh filename=package://aubo_description/meshes/aubo_i5l/s_Link.STL; visual mesh filename=package://aubo_description/meshes/aubo_i5l/s_Link.STL
- link shoulder_Link: geometry collision mesh filename=package://aubo_description/meshes/aubo_i5l/shoulder_Link.STL; visual mesh filename=package://aubo_description/meshes/aubo_i5l/shoulder_Link.STL
- link u_Link: geometry collision mesh filename=package://aubo_description/meshes/aubo_i5l/u_Link.STL; visual mesh filename=package://aubo_description/meshes/aubo_i5l/u_Link.STL
- link upperArm_Link: geometry collision mesh filename=package://aubo_description/meshes/aubo_i5l/upperArm_Link.STL; visual mesh filename=package://aubo_description/meshes/aubo_i5l/upperArm_Link.STL
- link w1_Link: geometry collision mesh filename=package://aubo_description/meshes/aubo_i5l/w1_Link.STL; visual mesh filename=package://aubo_description/meshes/aubo_i5l/w1_Link.STL
- link w2_Link: geometry collision mesh filename=package://aubo_description/meshes/aubo_i5l/w2_Link.STL; visual mesh filename=package://aubo_description/meshes/aubo_i5l/w2_Link.STL
- link wrist1_Link: geometry collision mesh filename=package://aubo_description/meshes/aubo_i5l/wrist1_Link.STL; visual mesh filename=package://aubo_description/meshes/aubo_i5l/wrist1_Link.STL
- link wrist2_Link: geometry collision mesh filename=package://aubo_description/meshes/aubo_i5l/wrist2_Link.STL; visual mesh filename=package://aubo_description/meshes/aubo_i5l/wrist2_Link.STL
- link wrist3_Link: geometry collision mesh filename=package://aubo_description/meshes/aubo_i5l/wrist3_Link.STL; visual mesh filename=package://aubo_description/meshes/aubo_i5l/wrist3_Link.STL

File: aubo_description/urdf/aubo_i5L.urdf.xacro (robot description, xacro)
@@ -17,5 +17,5 @@
       <origin rpy="0 0 0" xyz="0 0 0"/>
       <geometry>
-        <mesh filename="package://aubo_description/meshesL/base_link.STL"/>
+        <mesh filename="package://aubo_description/meshes/aubo_i5l/base_link.STL"/>
       </geometry>
        <material name="orange">
@@ -26,5 +26,5 @@
       <origin rpy="0 0 0" xyz="0 0 0"/>
       <geometry>
-        <mesh filename="package://aubo_description/meshesL/base_link.STL"/>
+        <mesh filename="package://aubo_description/meshes/aubo_i5l/base_link.STL"/>
       </geometry>
     </collision>
@@ -39,5 +39,5 @@
       <origin rpy="0 0 0" xyz="0 0 0"/>
       <geometry>
-        <mesh filename="package://aubo_description/meshesL/shoulder_Link.STL"/>
+        <mesh filename="package://aubo_description/meshes/aubo_i5l/shoulder_Link.STL"/>
       </geometry>
        <material name="orange">
@@ -48,5 +48,5 @@
       <origin rpy="0 0 0" xyz="0 0 0"/>
       <geometry>
-        <mesh filename="package://aubo_description/meshesL/shoulder_Link.STL"/>
+        <mesh filename="package://aubo_description/meshes/aubo_i5l/shoulder_Link.STL"/>
       </geometry>
     </collision>
@@ -68,5 +68,5 @@
       <origin rpy="0 0 0" xyz="0 0 0"/>
       <geometry>
-        <mesh filename="package://aubo_description/meshesL/upperArm_Link.STL"/>
+        <mesh filename="package://aubo_description/meshes/aubo_i5l/upperArm_Link.STL"/>
       </geometry>
        <material name="orange">
@@ -77,5 +77,5 @@
       <origin rpy="0 0 0" xyz="0 0 0"/>
       <geometry>
-        <mesh filename="package://aubo_description/meshesL/upperArm_Link.STL"/>
+        <mesh filename="package://aubo_description/meshes/aubo_i5l/upperArm_Link.STL"/>
       </geometry>
     </collision>
@@ -97,5 +97,5 @@
       <origin rpy="0 0 0" xyz="0 0 0"/>
       <geometry>
-        <mesh filename="package://aubo_description/meshesL/foreArm_Link.STL"/>
+        <mesh filename="package://aubo_description/meshes/aubo_i5l/foreArm_Link.STL"/>
       </geometry>
         <material name="orange">
@@ -106,5 +106,5 @@
       <origin rpy="0 0 0" xyz="0 0 0"/>
       <geometry>
-        <mesh filename="package://aubo_description/meshesL/foreArm_Link.STL"/>
+        <mesh filename="package://aubo_description/meshes/aubo_i5l/foreArm_Link.STL"/>
       </geometry>
     </collision>
@@ -126,5 +126,5 @@
       <origin rpy="0 0 0" xyz="0 0 0"/>
       <geometry>
-        <mesh filename="package://aubo_description/meshesL/wrist1_Link.STL"/>
+        <mesh filename="package://aubo_description/meshes/aubo_i5l/wrist1_Link.STL"/>
       </geometry>
      <material name="orange">
@@ -135,5 +135,5 @@
       <origin rpy="0 0 0" xyz="0 0 0"/>
       <geometry>
-        <mesh filename="package://aubo_description/meshesL/wrist1_Link.STL"/>
+        <mesh filename="package://aubo_description/meshes/aubo_i5l/wrist1_Link.STL"/>
       </geometry>
     </collision>
@@ -155,5 +155,5 @@
       <origin rpy="0 0 0" xyz="0 0 0"/>
       <geometry>
-        <mesh filename="package://aubo_description/meshesL/wrist2_Link.STL"/>
+        <mesh filename="package://aubo_description/meshes/aubo_i5l/wrist2_Link.STL"/>
       </geometry>
       <material name="orange">
@@ -164,5 +164,5 @@
       <origin rpy="0 0 0" xyz="0 0 0"/>
       <geometry>
-        <mesh filename="package://aubo_description/meshesL/wrist2_Link.STL"/>
+        <mesh filename="package://aubo_description/meshes/aubo_i5l/wrist2_Link.STL"/>
       </geometry>
     </collision>
@@ -184,14 +184,14 @@
       <origin rpy="0 0 0" xyz="0 0 0"/>
       <geometry>
-        <mesh filename="package://aubo_description/meshesL/wrist3_Link.STL"/>
-      </geometry>
-      <material name="black">
-        <color rgba="0.25098 0.25098 0.25098"/>
-      </material>
-    </visual>
-    <collision>
-      <origin rpy="0 0 0" xyz="0 0 0"/>
-      <geometry>
-        <mesh filename="package://aubo_description/meshesL/wrist3_Link.STL"/>
+        <mesh filename="package://aubo_description/meshes/aubo_i5l/wrist3_Link.STL"/>
+      </geometry>
+      <material name="black">
+        <color rgba="0.25098 0.25098 0.25098"/>
+      </material>
+    </visual>
+    <collision>
+      <origin rpy="0 0 0" xyz="0 0 0"/>
+      <geometry>
+        <mesh filename="package://aubo_description/meshes/aubo_i5l/wrist3_Link.STL"/>
       </geometry>
     </collision>
@@ -213,14 +213,14 @@
       <origin rpy="0 0 0" xyz="0 0 0"/>
       <geometry>
-        <mesh filename="package://aubo_description/meshesL/w2_Link.STL"/>
-      </geometry>
-      <material name="black">
-        <color rgba="0.25098 0.25098 0.25098"/>
-      </material>
-    </visual>
-    <collision>
-      <origin rpy="0 0 0" xyz="0 0 0"/>
-      <geometry>
-        <mesh filename="package://aubo_description/meshesL/w2_Link.STL"/>
+        <mesh filename="package://aubo_description/meshes/aubo_i5l/w2_Link.STL"/>
+      </geometry>
+      <material name="black">
+        <color rgba="0.25098 0.25098 0.25098"/>
+      </material>
+    </visual>
+    <collision>
+      <origin rpy="0 0 0" xyz="0 0 0"/>
+      <geometry>
+        <mesh filename="package://aubo_description/meshes/aubo_i5l/w2_Link.STL"/>
       </geometry>
     </collision>
@@ -241,14 +241,14 @@
       <origin rpy="0 0 0" xyz="0 0 0"/>
       <geometry>
-        <mesh filename="package://aubo_description/meshesL/w1_Link.STL"/>
-      </geometry>
-      <material name="black">
-        <color rgba="0.25098 0.25098 0.25098"/>
-      </material>
-    </visual>
-    <collision>
-      <origin rpy="0 0 0" xyz="0 0 0"/>
-      <geometry>
-        <mesh filename="package://aubo_description/meshesL/w1_Link.STL"/>
+        <mesh filename="package://aubo_description/meshes/aubo_i5l/w1_Link.STL"/>
+      </geometry>
+      <material name="black">
+        <color rgba="0.25098 0.25098 0.25098"/>
+      </material>
+    </visual>
+    <collision>
+      <origin rpy="0 0 0" xyz="0 0 0"/>
+      <geometry>
+        <mesh filename="package://aubo_description/meshes/aubo_i5l/w1_Link.STL"/>
       </geometry>
     </collision>
@@ -269,14 +269,14 @@
       <origin rpy="0 0 0" xyz="0 0 0"/>
       <geometry>
-        <mesh filename="package://aubo_description/meshesL/u_Link.STL"/>
-      </geometry>
-      <material name="black">
-        <color rgba="0.25098 0.25098 0.25098"/>
-      </material>
-    </visual>
-    <collision>
-      <origin rpy="0 0 0" xyz="0 0 0"/>
-      <geometry>
-        <mesh filename="package://aubo_description/meshesL/u_Link.STL"/>
+        <mesh filename="package://aubo_description/meshes/aubo_i5l/u_Link.STL"/>
+      </geometry>
+      <material name="black">
+        <color rgba="0.25098 0.25098 0.25098"/>
+      </material>
+    </visual>
+    <collision>
+      <origin rpy="0 0 0" xyz="0 0 0"/>
+      <geometry>
+        <mesh filename="package://aubo_description/meshes/aubo_i5l/u_Link.STL"/>
       </geometry>
     </collision>
@@ -297,14 +297,14 @@
       <origin rpy="0 0 0" xyz="0 0 0"/>
       <geometry>
-        <mesh filename="package://aubo_description/meshesL/f1_Link.STL"/>
-      </geometry>
-      <material name="black">
-        <color rgba="0.25098 0.25098 0.25098"/>
-      </material>
-    </visual>
-    <collision>
-      <origin rpy="0 0 0" xyz="0 0 0"/>
-      <geometry>
-        <mesh filename="package://aubo_description/meshesL/f1_Link.STL"/>
+        <mesh filename="package://aubo_description/meshes/aubo_i5l/f1_Link.STL"/>
+      </geometry>
+      <material name="black">
+        <color rgba="0.25098 0.25098 0.25098"/>
+      </material>
+    </visual>
+    <collision>
+      <origin rpy="0 0 0" xyz="0 0 0"/>
+      <geometry>
+        <mesh filename="package://aubo_description/meshes/aubo_i5l/f1_Link.STL"/>
       </geometry>
     </collision>
@@ -325,14 +325,14 @@
       <origin rpy="0 0 0" xyz="0 0 0"/>
       <geometry>
-        <mesh filename="package://aubo_description/meshesL/s_Link.STL"/>
-      </geometry>
-      <material name="black">
-        <color rgba="0.25098 0.25098 0.25098"/>
-      </material>
-    </visual>
-    <collision>
-      <origin rpy="0 0 0" xyz="0 0 0"/>
-      <geometry>
-        <mesh filename="package://aubo_description/meshesL/s_Link.STL"/>
+        <mesh filename="package://aubo_description/meshes/aubo_i5l/s_Link.STL"/>
+      </geometry>
+      <material name="black">
+        <color rgba="0.25098 0.25098 0.25098"/>
+      </material>
+    </visual>
+    <collision>
+      <origin rpy="0 0 0" xyz="0 0 0"/>
+      <geometry>
+        <mesh filename="package://aubo_description/meshes/aubo_i5l/s_Link.STL"/>
       </geometry>
     </collision>
