Commit message: add changelog

File: aubo_description/urdf/aubo_i5l.urdf.xacro (robot description, xacro)
@@ -7,5 +7,5 @@
   <xacro:include filename="$(find aubo_description)/urdf/aubo.transmission.xacro" />
   <xacro:include filename="$(find aubo_description)/urdf/aubo.gazebo.xacro" />
-  <xacro:include filename="$(find your_robot_description)/urdf/materials.xacro" />
+  <!--<xacro:include filename="$(find aubo_description)/urdf/materials.xacro" /> -->
   <link name="base_link">
     <inertial>
@@ -344,9 +344,9 @@
     <axis xyz="0 0 0"/>
   </joint>
-  <link name="world" />
+ <!-- <link name="world" />
   <joint name="world_joint" type="fixed">
     <parent link="world" />
     <child link = "base_link" />
     <origin xyz="0.0 0.0 0.0" rpy="0.0 0.0 0.0" />
-  </joint>
+  </joint> -->
 </robot>
