Commit message: add aubo_i10 control

File: aubo_description/urdf/aubo_i10.urdf (robot description, URDF)
Before this commit: robot aubo_i10, 7 links, 6 joints
Joints:
- joint foreArm_joint: axis 0 0 -1 -> 0 0 1

Commit message: test:Add melodic version of aubo_demo
In aubo_demo package, add the melodic version of the demo,
and use moveit to program and control the robot.

File: aubo_description/urdf/aubo_i10.urdf (robot description, URDF)
Before this commit: robot aubo_i10, 7 links, 6 joints
Joints:
- joint foreArm_joint: limit lower=-3.05 upper=3.05 effort=0 velocity=0 -> lower=-3.04 upper=3.04 effort=0 velocity=0
- joint shoulder_joint: limit lower=-3.05 upper=3.05 effort=0 velocity=0 -> lower=-3.04 upper=3.04 effort=0 velocity=0
- joint upperArm_joint: limit lower=-3.05 upper=3.05 effort=0 velocity=0 -> lower=-3.04 upper=3.04 effort=0 velocity=0
- joint wrist1_joint: limit lower=-3.05 upper=3.05 effort=0 velocity=0 -> lower=-3.04 upper=3.04 effort=0 velocity=0
- joint wrist2_joint: limit lower=-3.05 upper=3.05 effort=0 velocity=0 -> lower=-3.04 upper=3.04 effort=0 velocity=0
- joint wrist3_joint: limit lower=-3.05 upper=3.05 effort=0 velocity=0 -> lower=-3.04 upper=3.04 effort=0 velocity=0

File: aubo_description/urdf/aubo_i16.urdf (robot description, URDF)
Before this commit: robot aubo_i16, 8 links, 7 joints
Joints:
- joint foreArm_joint: limit lower=-3.05 upper=3.05 effort=0 velocity=0 -> lower=-3.04 upper=3.04 effort=0 velocity=0
- joint shoulder_joint: limit lower=-3.05 upper=3.05 effort=0 velocity=0 -> lower=-3.04 upper=3.04 effort=0 velocity=0
- joint upperArm_joint: limit lower=-3.05 upper=3.05 effort=0 velocity=0 -> lower=-3.04 upper=3.04 effort=0 velocity=0
- joint wrist1_joint: limit lower=-3.05 upper=3.05 effort=0 velocity=0 -> lower=-3.04 upper=3.04 effort=0 velocity=0
- joint wrist2_joint: limit lower=-3.05 upper=3.05 effort=0 velocity=0 -> lower=-3.04 upper=3.04 effort=0 velocity=0
- joint wrist3_joint: limit lower=-3.05 upper=3.05 effort=0 velocity=0 -> lower=-3.04 upper=3.04 effort=0 velocity=0

File: aubo_description/urdf/aubo_i3.urdf (robot description, URDF)
Before this commit: robot aubo_i3, 8 links, 7 joints
Joints:
- joint foreArm_joint: limit lower=-3.05 upper=3.05 effort=0 velocity=0 -> lower=-3.04 upper=3.04 effort=0 velocity=0
- joint shoulder_joint: limit lower=-3.05 upper=3.05 effort=0 velocity=0 -> lower=-3.04 upper=3.04 effort=0 velocity=0
- joint upperArm_joint: limit lower=-3.05 upper=3.05 effort=0 velocity=0 -> lower=-3.04 upper=3.04 effort=0 velocity=0
- joint wrist1_joint: limit lower=-3.05 upper=3.05 effort=0 velocity=0 -> lower=-3.04 upper=3.04 effort=0 velocity=0
- joint wrist2_joint: limit lower=-3.05 upper=3.05 effort=0 velocity=0 -> lower=-3.04 upper=3.04 effort=0 velocity=0
- joint wrist3_joint: limit lower=-3.05 upper=3.05 effort=0 velocity=0 -> lower=-3.04 upper=3.04 effort=0 velocity=0

File: aubo_description/urdf/aubo_i5.urdf (robot description, URDF)
Before this commit: robot aubo_i5, 8 links, 7 joints
Joints:
- joint foreArm_joint: limit lower=-3.05 upper=3.05 effort=0 velocity=0 -> lower=-3.04 upper=3.04 effort=0 velocity=0
- joint shoulder_joint: limit lower=-3.05 upper=3.05 effort=0 velocity=0 -> lower=-3.04 upper=3.04 effort=0 velocity=0
- joint upperArm_joint: limit lower=-3.05 upper=3.05 effort=0 velocity=0 -> lower=-3.04 upper=3.04 effort=0 velocity=0
- joint wrist1_joint: limit lower=-3.05 upper=3.05 effort=0 velocity=0 -> lower=-3.04 upper=3.04 effort=0 velocity=0
- joint wrist2_joint: limit lower=-3.05 upper=3.05 effort=0 velocity=0 -> lower=-3.04 upper=3.04 effort=0 velocity=0
- joint wrist3_joint: limit lower=-3.05 upper=3.05 effort=0 velocity=0 -> lower=-3.04 upper=3.04 effort=0 velocity=0

File: aubo_description/urdf/aubo_i5.urdf.xacro (robot description, xacro)
@@ -57,5 +57,5 @@
     <child link="shoulder_Link" />
     <axis xyz="0 0 1" />
-    <limit lower="-3.05" upper="3.05" effort="0" velocity="0" />
+    <limit lower="-3.04" upper="3.04" effort="0" velocity="0" />
   </joint>
   <link name="upperArm_Link">
@@ -86,5 +86,5 @@
     <child link="upperArm_Link" />
     <axis xyz="0 0 1" />
-    <limit lower="-3.05" upper="3.05" effort="0" velocity="0" />
+    <limit lower="-3.04" upper="3.04" effort="0" velocity="0" />
   </joint>
   <link name="foreArm_Link">
@@ -115,5 +115,5 @@
     <child link="foreArm_Link" />
     <axis xyz="0 0 1" />
-    <limit lower="-3.05" upper="3.05" effort="0" velocity="0" />
+    <limit lower="-3.04" upper="3.04" effort="0" velocity="0" />
   </joint>
   <link name="wrist1_Link">
@@ -144,5 +144,5 @@
     <child link="wrist1_Link" />
     <axis xyz="0 0 1" />
-    <limit lower="-3.05" upper="3.05" effort="0" velocity="0" />
+    <limit lower="-3.04" upper="3.04" effort="0" velocity="0" />
   </joint>
   <link name="wrist2_Link">
@@ -173,5 +173,5 @@
     <child link="wrist2_Link" />
     <axis xyz="0 0 1" />
-    <limit lower="-3.05" upper="3.05" effort="0" velocity="0" />
+    <limit lower="-3.04" upper="3.04" effort="0" velocity="0" />
   </joint>
   <link name="wrist3_Link">
@@ -202,5 +202,5 @@
     <child link="wrist3_Link" />
     <axis xyz="0 0 1" />
-    <limit lower="-3.05" upper="3.05" effort="0" velocity="0" />
+    <limit lower="-3.04" upper="3.04" effort="0" velocity="0" />
   </joint>
   <link name="world" />

File: aubo_description/urdf/aubo_i5L.urdf (robot description, URDF)
Before this commit: robot aubo_i5L_robot, 13 links, 12 joints
Joints:
- joint foreArm_joint: limit lower=-3.05 upper=3.05 effort=0 velocity=0 -> lower=-3.04 upper=3.04 effort=0 velocity=0
- joint shoulder_joint: limit lower=-3.05 upper=3.05 effort=0 velocity=0 -> lower=-3.04 upper=3.04 effort=0 velocity=0
- joint upperArm_joint: limit lower=-3.05 upper=3.05 effort=0 velocity=0 -> lower=-3.04 upper=3.04 effort=0 velocity=0
- joint wrist1_joint: limit lower=-3.05 upper=3.05 effort=0 velocity=0 -> lower=-3.04 upper=3.04 effort=0 velocity=0
- joint wrist2_joint: limit lower=-3.05 upper=3.05 effort=0 velocity=0 -> lower=-3.04 upper=3.04 effort=0 velocity=0
- joint wrist3_joint: limit lower=-3.05 upper=3.05 effort=0 velocity=0 -> lower=-3.04 upper=3.04 effort=0 velocity=0

File: aubo_description/urdf/aubo_i5l.urdf.xacro (robot description, xacro)
@@ -57,5 +57,5 @@
     <child link="shoulder_Link"/>
     <axis xyz="0 0 1"/>
-    <limit effort="0" lower="-3.05" upper="3.05" velocity="0"/>
+    <limit effort="0" lower="-3.04" upper="3.04" velocity="0"/>
   </joint>
   <link name="upperArm_Link">
@@ -86,5 +86,5 @@
     <child link="upperArm_Link"/>
     <axis xyz="0 0 1"/>
-    <limit effort="0" lower="-3.05" upper="3.05" velocity="0"/>
+    <limit effort="0" lower="-3.04" upper="3.04" velocity="0"/>
   </joint>
   <link name="foreArm_Link">
@@ -115,5 +115,5 @@
     <child link="foreArm_Link"/>
     <axis xyz="0 0 1"/>
-    <limit effort="0" lower="-3.05" upper="3.05" velocity="0"/>
+    <limit effort="0" lower="-3.04" upper="3.04" velocity="0"/>
   </joint>
   <link name="wrist1_Link">
@@ -144,5 +144,5 @@
     <child link="wrist1_Link"/>
     <axis xyz="0 0 1"/>
-    <limit effort="0" lower="-3.05" upper="3.05" velocity="0"/>
+    <limit effort="0" lower="-3.04" upper="3.04" velocity="0"/>
   </joint>
   <link name="wrist2_Link">
@@ -173,5 +173,5 @@
     <child link="wrist2_Link"/>
     <axis xyz="0 0 1"/>
-    <limit effort="0" lower="-3.05" upper="3.05" velocity="0"/>
+    <limit effort="0" lower="-3.04" upper="3.04" velocity="0"/>
   </joint>
   <link name="wrist3_Link">
@@ -202,5 +202,5 @@
     <child link="wrist3_Link"/>
     <axis xyz="0 0 1"/>
-    <limit effort="0" lower="-3.05" upper="3.05" velocity="0"/>
+    <limit effort="0" lower="-3.04" upper="3.04" velocity="0"/>
   </joint>
   <link name="w2_Link">
@@ -292,5 +292,5 @@
       <origin rpy="0 0 0" xyz="0.30397 -0.00049907 0.08414"/>
       <mass value="0.22341"/>
-      <inertia ixx="0.00030759" ixy="3.3453E-05" ixz="0.00029518" iyy="0.021935" iyz="-3.0561E-06" izz="0.022161"/>
+      <inertia ixx="0.00030759" ixy="3.3453E-05" ixz="0.00029518" iyy="0.021935" iyz="-3.0461E-06" izz="0.022161"/>
     </inertial>
     <visual>

File: aubo_description/urdf/aubo_i7.urdf (robot description, URDF)
Before this commit: robot aubo_i7, 8 links, 7 joints
Joints:
- joint foreArm_Joint: limit lower=-3.05 upper=3.05 effort=0 velocity=0 -> lower=-3.04 upper=3.04 effort=0 velocity=0
- joint shoulder_Joint: limit lower=-3.05 upper=3.05 effort=0 velocity=0 -> lower=-3.04 upper=3.04 effort=0 velocity=0
- joint upperArm_Joint: limit lower=-3.05 upper=3.05 effort=0 velocity=0 -> lower=-3.04 upper=3.04 effort=0 velocity=0
- joint wrist1_Joint: limit lower=-3.05 upper=3.05 effort=0 velocity=0 -> lower=-3.04 upper=3.04 effort=0 velocity=0
- joint wrist2_Joint: limit lower=-3.05 upper=3.05 effort=0 velocity=0 -> lower=-3.04 upper=3.04 effort=0 velocity=0
- joint wrist3_Joint: limit lower=-3.05 upper=3.05 effort=0 velocity=0 -> lower=-3.04 upper=3.04 effort=0 velocity=0

File: aubo_gazebo/urdf/aubo_i10.xacro (robot description, xacro)
@@ -148,5 +148,5 @@
     <child link="shoulder_Link" />
     <axis xyz="0 0 1" />
-    <limit lower="-3.05" upper="3.05" effort="1000" velocity="100" />
+    <limit lower="-3.04" upper="3.04" effort="1000" velocity="100" />
   </joint>
 <!--/////////////////////////////// UPPERARM_LINK ////////////////////////////////////-->
@@ -177,5 +177,5 @@
     <child link="upperArm_Link" />
     <axis xyz="0 0 1" />
-    <limit lower="-3.05" upper="3.05" effort="1000" velocity="100" />
+    <limit lower="-3.04" upper="3.04" effort="1000" velocity="100" />
   </joint>
 <!--/////////////////////////////// FOREARM_LINK ////////////////////////////////////-->
@@ -206,5 +206,5 @@
     <child link="foreArm_Link" />
     <axis xyz="0 0 1" />
-    <limit lower="-3.05" upper="3.05" effort="1000" velocity="100" />
+    <limit lower="-3.04" upper="3.04" effort="1000" velocity="100" />
   </joint>
 <!--/////////////////////////////// WRIST1_LINK ////////////////////////////////////-->
@@ -235,5 +235,5 @@
     <child link="wrist1_Link" />
     <axis xyz="0 0 1" />
-    <limit lower="-3.05" upper="3.05" effort="1000" velocity="100" />
+    <limit lower="-3.04" upper="3.04" effort="1000" velocity="100" />
   </joint>
 <!--/////////////////////////////// WRIST2_LINK ////////////////////////////////////-->
@@ -264,5 +264,5 @@
     <child link="wrist2_Link" />
     <axis xyz="0 0 1" />
-    <limit lower="-3.05" upper="3.05" effort="1000" velocity="100" />
+    <limit lower="-3.04" upper="3.04" effort="1000" velocity="100" />
   </joint>
 <!--/////////////////////////////// WRIST3_LINK ////////////////////////////////////-->
@@ -293,5 +293,5 @@
     <child link="wrist3_Link" />
     <axis xyz="0 0 1" />
-    <limit lower="-3.05" upper="3.05" effort="1000" velocity="100" />
+    <limit lower="-3.04" upper="3.04" effort="1000" velocity="100" />
   </joint>
  <!--/////////////////////////////// WORLD ////////////////////////////////////-->

File: aubo_gazebo/urdf/aubo_i3.xacro (robot description, xacro)
@@ -148,5 +148,5 @@
     <child link="shoulder_Link" />
     <axis xyz="0 0 1" />
-    <limit lower="-3.05" upper="3.05" effort="300" velocity="100" />
+    <limit lower="-3.04" upper="3.04" effort="300" velocity="100" />
   </joint>
  <!--/////////////////////////////// UPPERARM_LINK ////////////////////////////////////-->
@@ -177,5 +177,5 @@
     <child link="upperArm_Link" />
     <axis xyz="0 0 1" />
-    <limit lower="-3.05" upper="3.05" effort="300" velocity="100" />
+    <limit lower="-3.04" upper="3.04" effort="300" velocity="100" />
   </joint>
  <!--/////////////////////////////// FOREARM_LINK ////////////////////////////////////-->
@@ -206,5 +206,5 @@
     <child link="foreArm_Link" />
     <axis xyz="0 0 1" />
-    <limit lower="-3.05" upper="3.05" effort="300" velocity="100" />
+    <limit lower="-3.04" upper="3.04" effort="300" velocity="100" />
   </joint>
  <!--/////////////////////////////// WRIST1_LINK ////////////////////////////////////-->
@@ -235,5 +235,5 @@
     <child link="wrist1_Link" />
     <axis xyz="0 0 1" />
-    <limit lower="-3.05" upper="3.05" effort="300" velocity="100" />
+    <limit lower="-3.04" upper="3.04" effort="300" velocity="100" />
   </joint>
 <!--/////////////////////////////// WRIST2_LINK ////////////////////////////////////-->
@@ -264,5 +264,5 @@
     <child  link="wrist2_Link" />
     <axis xyz="0 0 1" />
-    <limit lower="-3.05" upper="3.05" effort="300" velocity="100" />
+    <limit lower="-3.04" upper="3.04" effort="300" velocity="100" />
   </joint>
 <!--/////////////////////////////// WRIST3_LINK ////////////////////////////////////-->
@@ -293,5 +293,5 @@
     <child link="wrist3_Link" />
     <axis xyz="0 0 1" />
-    <limit lower="-3.05" upper="3.05" effort="300" velocity="100" />
+    <limit lower="-3.04" upper="3.04" effort="300" velocity="100" />
   </joint>
  <!--/////////////////////////////// WORLD ////////////////////////////////////-->

File: aubo_gazebo/urdf/aubo_i5.xacro (robot description, xacro)
@@ -136,5 +136,5 @@
     <child link="shoulder_Link" />
     <axis xyz="0 0 1" />
-    <limit lower="-3.05" upper="3.05" effort="300" velocity="100" />
+    <limit lower="-3.04" upper="3.04" effort="300" velocity="100" />
   </joint>
   <!--/////////////////////////////// UPPERARM_LINK ////////////////////////////////////-->
@@ -165,5 +165,5 @@
     <child link="upperArm_Link" />
     <axis xyz="0 0 1" />
-    <limit lower="-3.05" upper="3.05" effort="300" velocity="100" />
+    <limit lower="-3.04" upper="3.04" effort="300" velocity="100" />
   </joint>
   <!--/////////////////////////////// FOREARM_LINK ////////////////////////////////////-->
@@ -194,5 +194,5 @@
     <child link="foreArm_Link" />
     <axis xyz="0 0 1" />
-    <limit lower="-3.05" upper="3.05" effort="300" velocity="100" />
+    <limit lower="-3.04" upper="3.04" effort="300" velocity="100" />
   </joint>
   <!--/////////////////////////////// WRIST1_LINK ////////////////////////////////////-->
@@ -223,5 +223,5 @@
     <child link="wrist1_Link" />
     <axis xyz="0 0 1" />
-    <limit lower="-3.05" upper="3.05" effort="300" velocity="100" />
+    <limit lower="-3.04" upper="3.04" effort="300" velocity="100" />
   </joint>
   <!--/////////////////////////////// WRIST2_LINK ////////////////////////////////////-->
@@ -252,5 +252,5 @@
     <child link="wrist2_Link" />
     <axis xyz="0 0 1" />
-    <limit lower="-3.05" upper="3.05" effort="300" velocity="100" />
+    <limit lower="-3.04" upper="3.04" effort="300" velocity="100" />
   </joint>
   <!--/////////////////////////////// WRIST3_LINK ////////////////////////////////////-->
@@ -281,5 +281,5 @@
     <child link="wrist3_Link" />
     <axis xyz="0 0 1" />
-    <limit lower="-3.05" upper="3.05" effort="300" velocity="100" />
+    <limit lower="-3.04" upper="3.04" effort="300" velocity="100" />
   </joint>
   <!-- /////////////////////////////////   i5 pedestal_Link   ////////////////////////////////////// -->
