Commit message: remove gripper from robot urdf

File: aubo_gazebo/urdf/aubo_i5.xacro (robot description, xacro)
@@ -19,9 +19,4 @@
     <!-- Constants -->
     <xacro:property name="M_PI" value="3.14159"/>
-    <xacro:property name="endEffectorPoleLength" value="0.325"/>
-    <xacro:property name="endEffectorPoleRadius" value="0.007"/>
-    <xacro:property name="endEffectorBoxLength" value="0.09"/>
-    <xacro:property name="endEffectorBoxWidth" value="0.130"/>
-    <xacro:property name="endEffectorBoxHeight" value="0.080"/>
     <!--/////////////////// DYNAMICS PARAM //////////////////////-->
     <xacro:macro name="I5_Shoulder_Inertia">
@@ -81,15 +76,4 @@
     </xacro:macro>
     <xacro:macro name="I5_Wrist3_Inertia">
-        <origin xyz="0.0 0.0 -0.0071"
-                rpy="0 0 0" />
-        <mass value="0.40" />
-        <inertia ixx="0.013939"
-                 ixy="0"
-                 ixz="0"
-                 iyy="0.013988"
-                 iyz="0.0"
-                 izz="0.0224092" />
-    </xacro:macro>
-    <xacro:macro name="I5_End_Effector_Inertia">
         <origin xyz="0.0 0.0 -0.0071"
                 rpy="0 0 0" />
@@ -298,42 +282,4 @@
     <axis xyz="0 0 1" />
     <limit lower="-3.05" upper="3.05" effort="300" velocity="100" />
-  </joint>
-    <!--/////////////////////////////// END_EFFECTOR_LINK ////////////////////////////////////-->
-  <link name="end_effector_Link">
-    <inertial>
-      <xacro:I5_End_Effector_Inertia />
-    </inertial>
-    <visual>
-      <origin xyz="0 0 ${endEffectorPoleLength/2}" rpy="0 0 0" />
-      <geometry>
-        <!-- <mesh filename="package://harvester_description/meshes/end_effector.DAE" /> -->
-      <cylinder length="${endEffectorPoleLength}" radius="${endEffectorPoleRadius}"/>
-      </geometry>
-      <material name="">
-        <color rgba="1 1 1 1" />
-      </material>
-    </visual>
-    <visual>
-      <origin xyz="0 0 ${endEffectorBoxLength/2}" rpy="0 0 0"/>
-      <geometry>
-        <box size="${endEffectorBoxWidth} ${endEffectorBoxHeight} ${endEffectorBoxLength}"/>
-      </geometry>
-      <material name="">
-        <color rgba="1 1 1 1" />
-      </material>
-    </visual>
-    <collision>
-      <origin xyz="0 0 ${endEffectorPoleLength/2}" rpy="0 0 0" />
-      <geometry>
-        <!-- <mesh filename="package://harvester_description/meshes/end_effector_new.STL" /> -->
-      <cylinder length="${endEffectorPoleLength}" radius="${endEffectorPoleRadius}"/>
-      </geometry>
-    </collision>
-  </link>
-  <!--/////////////////////////////// END_EFFECTOR_JOINT ////////////////////////////////////-->
-  <joint name="end_effector_joint" type="fixed">
-    <origin xyz="0.0 0.0 0.0" rpy="0.0 0.0 0.0" />
-    <parent link="wrist3_Link" />
-    <child link="end_effector_Link" />
   </joint>
   <!-- /////////////////////////////////   i5 pedestal_Link   ////////////////////////////////////// -->
@@ -357,9 +303,10 @@
     <origin xyz="0.0 0.0 0.1" rpy="0.0 0.0 0.0" />
   </joint> -->
+ <!-- /////////////////////////////////   burro bed   ////////////////////////////////////// -->
   <joint name="base_link_joint" type="fixed">
     <parent link="bed" />
     <child link ="base_link" />
     <origin xyz="0 0 0" rpy="0 0 0" />
-  </joint> -->
+  </joint>
   <!-- /////////////////////////////////   gazebo color   ////////////////////////////////////// -->
   <!-- <gazebo reference="pedestal_Link">

Commit message: remove burro_bad-base link connection:

File: aubo_gazebo/urdf/aubo_i5.xacro (robot description, xacro)
@@ -303,10 +303,4 @@
     <origin xyz="0.0 0.0 0.1" rpy="0.0 0.0 0.0" />
   </joint> -->
- <!-- /////////////////////////////////   burro bed   ////////////////////////////////////// -->
-  <joint name="base_link_joint" type="fixed">
-    <parent link="bed" />
-    <child link ="base_link" />
-    <origin xyz="0 0 0" rpy="0 0 0" />
-  </joint>
   <!-- /////////////////////////////////   gazebo color   ////////////////////////////////////// -->
   <!-- <gazebo reference="pedestal_Link">
