Commit message: Fix:Error that E5 robot cannot be simulated in gazebo

File: aubo_gazebo/urdf/aubo_e5.xacro (robot description, xacro)
@@ -20,115 +20,6 @@
     <xacro:property name="M_PI" value="3.14159"/>
     <!--/////////////////// DYNAMICS PARAM //////////////////////-->
-    <xacro:macro name="I5_Shoulder_Inertia">
-        <origin xyz="0.0 0.006 -0.002"
-                rpy="0 0 0" />
-        <mass value="5.05" />
-        <inertia ixx="0.0148"
-                 ixy="0"
-                 ixz="0"
-                 iyy="0.0143"
-                 iyz="-0.0"
-                 izz="0.0095" />
-    </xacro:macro>
-    <xacro:macro name="I5_UpperArm_Inertia">
-        <origin xyz="0.304 0.0 -0.03"
-                rpy="0 0 0" />
-        <mass value="11.90" />
-        <inertia ixx="0.0305"
-                 ixy="0"
-                 ixz="0"
-                 iyy="0.4505"
-                 iyz="0"
-                 izz="0.0095" />
-    </xacro:macro>
-    <xacro:macro name="I5_ForeArm_Inertia">
-        <origin xyz="0.415 0.0 0.0992"
-                rpy="0 0 0" />
-        <mass  value="3.3" />
-        <inertia ixx="0.0033"
-                 ixy="0"
-                 ixz="0.0009"
-                 iyy="0.0575"
-                 iyz="0"
-                 izz="0.0565" />
-    </xacro:macro>
-    <xacro:macro name="I5_Wrist1_Inertia">
-        <origin xyz="0.0 0.0028 -0.003"
-                rpy="0 0 0" />
-        <mass value="1.62" />
-        <inertia ixx="0.0023"
-                 ixy="0"
-                 ixz="0"
-                 iyy="0.0013"
-                 iyz="0.0"
-                 izz="0.0022" />
-    </xacro:macro>
-    <xacro:macro name="I5_Wrist2_Inertia">
-        <origin xyz="0.0 -0.0028 -0.003"
-                rpy="0 0 0" />
-        <mass value="1.62" />
-        <inertia ixx="0.0023"
-                 ixy="0"
-                 ixz="0"
-                 iyy="0.0013"
-                 iyz="0.0"
-                 izz="0.0022" />
-    </xacro:macro>
-    <xacro:macro name="I5_Wrist3_Inertia">
-        <origin xyz="0.0 0.0 -0.0071"
-                rpy="0 0 0" />
-        <mass value="0.40" />
-        <inertia ixx="0.013939"
-                 ixy="0"
-                 ixz="0"
-                 iyy="0.013988"
-                 iyz="0.0"
-                 izz="0.0224092" />
-    </xacro:macro>
-    <!--/////////////////////////////// BASE_LINK ////////////////////////////////////-->
-   <link
-    name="base_link">
-    <inertial>
-      <origin
-        xyz="4.2454E-05 -1.2043E-08 0.020702"
-        rpy="0 0 0" />
-      <mass
-        value="0.80619" />
-      <inertia
-        ixx="0.0013215"
-        ixy="2.5362E-09"
-        ixz="-1.4252E-05"
-        iyy="0.0013301"
-        iyz="-1.0084E-10"
-        izz="0.0023301" />
-    </inertial>
-    <visual>
-      <origin
-        xyz="0 0 0"
-        rpy="0 0 0" />
-      <geometry>
-        <mesh
-          filename="package://aubo_description/meshes/aubo_e5/visual/base_link.DAE" />
-      </geometry>
-      <material
-        name="">
-        <color
-          rgba="1 1 1 1" />
-      </material>
-    </visual>
-    <collision>
-      <origin
-        xyz="0 0 0"
-        rpy="0 0 0" />
-      <geometry>
-        <mesh
-          filename="package://aubo_description/meshes/aubo_e5/collision/base_link.STL" />
-      </geometry>
-    </collision>
-  </link>
-  <link
-    name="shoulder_Link">
-    <inertial>
-      <origin
+    <xacro:macro name="E5_Shoulder_Inertia">
+        <origin
         xyz="-2.1059E-08 0.0083051 0.065103"
         rpy="0 0 0" />
@@ -142,51 +33,7 @@
         iyz="-0.00021308"
         izz="0.0031979" />
-    </inertial>
-    <visual>
-      <origin
-        xyz="0 0 0"
-        rpy="0 0 0" />
-      <geometry>
-        <mesh
-          filename="package://aubo_description/meshes/aubo_e5/visual/shoulder_Link.DAE" />
-      </geometry>
-      <material
-        name="">
-        <color
-          rgba="1 1 1 1" />
-      </material>
-    </visual>
-    <collision>
-      <origin
-        xyz="0 0 0"
-        rpy="0 0 0" />
-      <geometry>
-        <mesh
-          filename="package://aubo_description/meshes/aubo_e5/collision/shoulder_Link.STL" />
-      </geometry>
-    </collision>
-  </link>
-  <joint
-    name="shoulder_joint"
-    type="revolute">
-    <origin
-      xyz="0 0 0.0495"
-      rpy="0 0 -3.1234" />
-    <parent
-      link="base_link" />
-    <child
-      link="shoulder_Link" />
-    <axis
-      xyz="0 0 1" />
-    <limit
-      lower="-3.05"
-      upper="3.05"
-      effort="0"
-      velocity="0" />
-  </joint>
-  <link
-    name="upperArm_Link">
-    <inertial>
-      <origin
+    </xacro:macro>
+    <xacro:macro name="E5_UpperArm_Inertia">
+       <origin
         xyz="0.204 -0.00063844 0.057604"
         rpy="0 0 0" />
@@ -200,51 +47,7 @@
         iyz="-4.6361E-06"
         izz="0.020135" />
-    </inertial>
-    <visual>
-      <origin
-        xyz="0 0 0"
-        rpy="0 0 0" />
-      <geometry>
-        <mesh
-          filename="package://aubo_description/meshes/aubo_e5/visual/upperArm_Link.DAE" />
-      </geometry>
-      <material
-        name="">
-        <color
-          rgba="1 1 1 1" />
-      </material>
-    </visual>
-    <collision>
-      <origin
-        xyz="0 0 0"
-        rpy="0 0 0" />
-      <geometry>
-        <mesh
-          filename="package://aubo_description/meshes/aubo_e5/collision/upperArm_Link.STL" />
-      </geometry>
-    </collision>
-  </link>
-  <joint
-    name="upperArm_joint"
-    type="revolute">
-    <origin
-      xyz="0 0.0786 0.0708"
-      rpy="-1.5708 -1.5708 0" />
-    <parent
-      link="shoulder_Link" />
-    <child
-      link="upperArm_Link" />
-    <axis
-      xyz="0 0 1" />
-    <limit
-      lower="-3.05"
-      upper="3.05"
-      effort="0"
-      velocity="0" />
-  </joint>
-  <link
-    name="foreArm_Link">
-    <inertial>
-      <origin
+    </xacro:macro>
+    <xacro:macro name="E5_ForeArm_Inertia">
+        <origin
         xyz="0.18368 0.00064681 0.055339"
         rpy="0 0 0" />
@@ -258,51 +61,7 @@
         iyz="-1.3488E-06"
         izz="0.0089876" />
-    </inertial>
-    <visual>
-      <origin
-        xyz="0 0 0"
-        rpy="0 0 0" />
-      <geometry>
-        <mesh
-          filename="package://aubo_description/meshes/aubo_e5/visual/foreArm_Link.DAE" />
-      </geometry>
-      <material
-        name="">
-        <color
-          rgba="1 1 1 1" />
-      </material>
-    </visual>
-    <collision>
-      <origin
-        xyz="0 0 0"
-        rpy="0 0 0" />
-      <geometry>
-        <mesh
-          filename="package://aubo_description/meshes/aubo_e5/collision/foreArm_Link.STL" />
-      </geometry>
-    </collision>
-  </link>
-  <joint
-    name="foreArm_joint"
-    type="revolute">
-    <origin
-      xyz="0.408 -0.0012767 0.0002"
-      rpy="3.1416 0 0" />
-    <parent
-      link="upperArm_Link" />
-    <child
-      link="foreArm_Link" />
-    <axis
-      xyz="0 0 1" />
-    <limit
-      lower="-3.05"
-      upper="3.05"
-      effort="0"
-      velocity="0" />
-  </joint>
-  <link
-    name="wrist1_Link">
-    <inertial>
-      <origin
+    </xacro:macro>
+    <xacro:macro name="E5_Wrist1_Inertia">
+        <origin
         xyz="-5.5568E-06 0.006024 0.051377"
         rpy="0 0 0" />
@@ -316,51 +75,7 @@
         iyz="-3.1316E-05"
         izz="0.00038517" />
-    </inertial>
-    <visual>
-      <origin
-        xyz="0 0 0"
-        rpy="0 0 0" />
-      <geometry>
-        <mesh
-          filename="package://aubo_description/meshes/aubo_e5/visual/wrist1_Link.DAE" />
-      </geometry>
-      <material
-        name="">
-        <color
-          rgba="1 1 1 1" />
-      </material>
-    </visual>
-    <collision>
-      <origin
-        xyz="0 0 0"
-        rpy="0 0 0" />
-      <geometry>
-        <mesh
-          filename="package://aubo_description/meshes/aubo_e5/collision/wrist1_Link.STL" />
-      </geometry>
-    </collision>
-  </link>
-  <joint
-    name="wrist1_joint"
-    type="revolute">
-    <origin
-      xyz="0.3736 -8.9586E-05 0.015624"
-      rpy="3.1415 0.03325 1.5708" />
-    <parent
-      link="foreArm_Link" />
-    <child
-      link="wrist1_Link" />
-    <axis
-      xyz="0 0 1" />
-    <limit
-      lower="-3.05"
-      upper="3.05"
-      effort="0"
-      velocity="0" />
-  </joint>
-  <link
-    name="wrist2_Link">
-    <inertial>
-      <origin
+    </xacro:macro>
+    <xacro:macro name="E5_Wrist2_Inertia">
+        <origin
         xyz="-0.00026766 -0.006018 0.051777"
         rpy="0 0 0" />
@@ -374,51 +89,7 @@
         iyz="3.1286E-05"
         izz="0.00038517" />
-    </inertial>
-    <visual>
-      <origin
-        xyz="0 0 0"
-        rpy="0 0 0" />
-      <geometry>
-        <mesh
-          filename="package://aubo_description/meshes/aubo_e5/visual/wrist2_Link.DAE" />
-      </geometry>
-      <material
-        name="">
-        <color
-          rgba="1 1 1 1" />
-      </material>
-    </visual>
-    <collision>
-      <origin
-        xyz="0 0 0"
-        rpy="0 0 0" />
-      <geometry>
-        <mesh
-          filename="package://aubo_description/meshes/aubo_e5/collision/wrist2_Link.STL" />
-      </geometry>
-    </collision>
-  </link>
-  <joint
-    name="wrist2_joint"
-    type="revolute">
-    <origin
-      xyz="-4.4976E-05 0.0438 0.0576"
-      rpy="-1.5708 0.03325 0.0010269" />
-    <parent
-      link="wrist1_Link" />
-    <child
-      link="wrist2_Link" />
-    <axis
-      xyz="0 0 1" />
-    <limit
-      lower="-3.05"
-      upper="3.05"
-      effort="0"
-      velocity="0" />
-  </joint>
-  <link
-    name="wrist3_Link">
-    <inertial>
-      <origin
+    </xacro:macro>
+    <xacro:macro name="E5_Wrist3_Inertia">
+        <origin
         xyz="3.5297E-07 0.00012801 -0.019327"
         rpy="0 0 0" />
@@ -432,46 +103,201 @@
         iyz="1.8269E-08"
         izz="0.00010284" />
-    </inertial>
-    <visual>
-      <origin
-        xyz="0 0 0"
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